File: provisioner/hexpansion_provisioner.kicad_pcb (KiCad board)
At the start: 2 copper layers, 100 x 37 mm, 29 parts, among them J1 Conn_02x10_Counter_Clockwise, J2 Conn_01x10_Pin, J3 Conn_01x05_Pin, J4 Conn_01x02_Pin, J5 Conn_01x04_Pin, SW1 SW_SPDT, U1 FT232H Breakout, U2 74LVC1G04, U3 MT9700

Commit message: Add pcb arwork and prep for manufacture.
Other:
- board text added: "r1.0"
